Commit message: Add ros2_control hardware interface, controller config, and Jacobian node scaffold
- Add gz_ros2_control Gazebo plugin to xacro
- Add ros2_control hardware block with velocity interfaces for leg joints
- Add controllers.yaml with JointStateBroadcaster and JointGroupVelocityController
- Update gazebo.launch.py to spawn controllers with timer delay
- Add th_rhex_control Python package with Jacobian velocity controller node

File: src/th_rhex_description/urdf/th_rhex.urdf.xacro (robot description, xacro)
@@ -5,4 +5,46 @@
 <robot
   name="th_rhex">
+  <!-- Gazebo ros2_control plugin -->
+  <gazebo>
+    <plugin filename="gz_ros2_control-system"
+      name="gz_ros2_control::GazeboSimROS2ControlPlugin">
+      <parameters>$(find th_rhex_description)/config/controllers.yaml</parameters>
+    </plugin>
+  </gazebo>
+  <!--ros2_control hardware interface-->
+  <ros2_control name="GazeboSystem" type="system">
+    <hardware>
+      <plugin>gz_ros2_control/GazeboSimSystem</plugin>
+    </hardware>
+    <!-- Acutated leg joint - velocity commanded-->
+    <joint name="fr_leg_joint">
+      <command_interface name="velocity"/>
+      <state_interface name="position"/>
+      <state_interface name="velocity"/>
+    </joint>
+    <joint name="ml_leg_joint">
+      <command_interface name="velocity"/>
+      <state_interface name="position"/>
+      <state_interface name="velocity"/>
+    </joint>
+    <joint name="rr_leg_joint">
+      <command_interface name="velocity"/>
+      <state_interface name="position"/>
+      <state_interface name="velocity"/>
+    </joint>
+    <!-- Passive wheel joints - state only-->
+    <joint name="fr_wheel_joint">
+      <state_interface name="position"/>
+      <state_interface name="velocity"/>
+    </joint>
+    <joint name="ml_wheel_joint">
+      <state_interface name="position"/>
+      <state_interface name="velocity"/>
+    </joint>
+    <joint name="rr_wheel_joint">
+      <state_interface name="position"/>
+      <state_interface name="velocity"/>
+    </joint>
+  </ros2_control>
   <link
     name="base_footprint" />
