Commit message: Replace th_rhex_description with separate 3-leg and 6-leg packages
- Add th_rhex_description_3leg and th_rhex_description_6leg packages
  with updated SolidWorks v2/v1 URDF exports
- Inject ros2_control hardware interface block into both URDFs
- Fix leg joint axes (ml, rr: 0 0 -1 → 0 0 1) for correct CCW rotation
- Rewrite gazebo.launch.py: resolve package:// → file://, $(find) →
  abs path, add /clock bridge, set use_sim_time=True
- Add Gazebo Harmonic-compatible minimal_world.sdf (inline ground plane)
- Add ros-jazzy-ros2-control/controllers/gz-ros2-control to Dockerfile

File: src/th_rhex_description_3leg/urdf/th_rhex.urdf.xacro (robot description, xacro)
@@ -3,6 +3,5 @@
      Commit Version: 1.6.0-4-g7f85cfe  Build Version: 1.6.7995.38578
      For more information, please see http://wiki.ros.org/sw_urdf_exporter -->
-<robot
-  name="th_rhex">
+<robot name="th_rhex">
   <!-- Gazebo ros2_control plugin -->
   <gazebo>
@@ -12,10 +11,8 @@
     </plugin>
   </gazebo>
-  <!--ros2_control hardware interface-->
   <ros2_control name="GazeboSystem" type="system">
     <hardware>
       <plugin>gz_ros2_control/GazeboSimSystem</plugin>
     </hardware>
-    <!-- Acutated leg joint - velocity commanded-->
     <joint name="fr_leg_joint">
       <command_interface name="velocity"/>
@@ -33,5 +30,4 @@
       <state_interface name="velocity"/>
     </joint>
-    <!-- Passive wheel joints - state only-->
     <joint name="fr_wheel_joint">
       <state_interface name="position"/>
@@ -246,17 +242,13 @@
     </collision>
   </link>
-  <joint
-    name="ml_leg_joint"
-    type="continuous">
-    <origin
-      xyz="2.3837470348731E-05 0.120249997292873 -0.016177780946989"
-      rpy="1.5707963267949 1.5707963267949 0" />
-    <parent
-      link="base_link" />
-    <child
-      link="ml_leg_link" />
-    <axis
-      xyz="0 0 -1" />
-  </joint>
+<!-- ml_leg_joint — keep current RPY, fix axis -->
+<joint name="ml_leg_joint" type="continuous">
+  <origin
+    xyz="2.3837470348731E-05 0.120249997292873 -0.016177780946989"
+    rpy="-1.5707963267949 1.25162281280328 -3.14159265358979"/>
+  <parent link="base_link"/>
+  <child link="ml_leg_link"/>
+  <axis xyz="-0.307748 0.915594 0.258804"/>
+</joint>
   <link
     name="ml_wheel_link">
@@ -304,5 +296,5 @@
     <origin
       xyz="0.0579914102340645 0.0191645608875115 0"
-      rpy="1.8899702911568 1.5707963267949 0" />
+      rpy="-1.5707963267949 0 0.319173513991623" />
     <parent
       link="ml_leg_link" />
@@ -352,17 +344,13 @@
     </collision>
   </link>
-  <joint
-    name="rr_leg_joint"
-    type="continuous">
-    <origin
-      xyz="-0.102853319292588 -0.0812499972928725 -0.0162297985657852"
-      rpy="1.5707963267949 1.5707963267949 0" />
-    <parent
-      link="base_link" />
-    <child
-      link="rr_leg_link" />
-    <axis
-      xyz="0 0 -1" />
-  </joint>
+<!-- rr_leg_joint — keep current RPY, fix axis -->
+<joint name="rr_leg_joint" type="continuous">
+  <origin
+    xyz="-0.102853319292588 -0.0812499972928725 -0.0162297985657852"
+    rpy="1.5707963267949 1.5707963267949 0"/>
+  <parent link="base_link"/>
+  <child link="rr_leg_link"/>
+  <axis xyz="-0.004909 -0.258828 -0.965911"/>
+</joint>
   <link
     name="rr_wheel_link">
